File: KiCad-d-pdm/KiCad-Diynamic-Project-Display-Module.kicad_sch (KiCad schematic)
At the start: 40 parts, among them SW1 SW_Push, SW10 SW_Push, SW11 SW_Push, SW12 SW_Push, SW13 SW_Push, SW14 SW_Push, SW15 SW_Push, SW16 SW_Push, SW17 RotaryEncoder_Switch_MP, SW18 RotaryEncoder_Switch_MP, SW2 SW_Push, SW3 SW_Push, SW4 SW_Push, SW5 SW_Push, SW6 SW_Push, SW7 SW_Push, SW8 SW_Push, SW9 SW_Push, U1 XIAO-RP2040-DIP

Commit message: Prodjekt
Parts:
- added Brd1: GME12864_OLED, OLED:SSD1306-0.91-OLED-4pin-128x32, symbol OLED:GME12864_OLED
- added D22, D23, D24, D25, D26, D27, D28, D29, D30, D31, D32, D33, D34, D35, D36, D37, D38, D39: D, Diode_SMD:D_SOD-123, symbol Device:D
- added J1: Conn_01x03_Pin, Connector_PinHeader_2.54mm:PinHeader_1x03_P2.54mm_Horizontal, symbol Connector:Conn_01x03_Pin
- added J2: Conn_01x02_Pin, Connector_PinHeader_2.54mm:PinHeader_1x02_P2.54mm_Horizontal, symbol Connector:Conn_01x02_Pin
- added R1, R2, R3, R4, R5: 200R, Resistor_SMD:R_0805_2012Metric_Pad1.20x1.40mm_HandSolder, symbol Device:R
- added U3: MCP23017_SO, Package_SO:SOIC-28W_7.5x17.9mm_P1.27mm, symbol Interface_Expansion:MCP23017_SO
- D18, D19, D20, D21: footprint (none) -> LED_THT:LED_D5.0mm
- SW1, SW10, SW11, SW12, SW13, SW14, SW15, SW16, SW2, SW3, SW4, SW5, SW6, SW7, SW8, SW9: footprint (none) -> Button_Switch_Keyboard:SW_Cherry_MX_1.00u_PCB
- SW17, SW18: footprint (none) -> Rotary_Encoder:RotaryEncoder_Alps_EC11E-Switch_Vertical_H20mm_MountingHoles
- U1: footprint Module:MOUDLE14P-XIAO-DIP-SMD -> OPL:XIAO-RP2040-DIP
Connections:
- net +5V: now also D1.4 (VDD), D10.4 (VDD), D11.4 (VDD), D12.4 (VDD), D13.4 (VDD), D14.4 (VDD), D15.4 (VDD), D16.4 (VDD), D2.4 (VDD), D3.4 (VDD), D4.4 (VDD), D5.4 (VDD), D6.4 (VDD), D7.4 (VDD), D8.4 (VDD), D9.4 (VDD), U3.18 (~{RESET}), U3.9 (VDD)
- net GND: now also D1.2 (VSS), D10.2 (VSS), D11.2 (VSS), D12.2 (VSS), D13.2 (VSS), D14.2 (VSS), D15.2 (VSS), D16.2 (VSS), D17.1 (K), D18.1 (K), D19.1 (K), D2.2 (VSS), D20.1 (K), D21.1 (K), D3.2 (VSS), D4.2 (VSS), D5.2 (VSS), D6.2 (VSS), D7.2 (VSS), D8.2 (VSS), D9.2 (VSS), SW17.C, SW18.C, Brd1.2 (GND), U3.10 (VSS), U3.15 (A0), U3.16 (A1), U3.17 (A2)
- net at D15.1 (DOUT): now also D16.3 (DIN)
- net at D15.3 (DIN): now also D14.1 (DOUT)
- net at D10.1 (DOUT): now also D11.3 (DIN)
- net at D10.3 (DIN): now also D9.1 (DOUT)
- net at D7.1 (DOUT): now also D8.3 (DIN)
- net at D7.3 (DIN): now also D6.1 (DOUT)
- net SW17.A: now reaches SW17.A
- net SW17.A: now also U3.23 (GPA2)
- net SW17.B: now reaches SW17.B
- net SW17.B: now also U3.24 (GPA3)
- net SW17.S: now reaches SW17.S1
- net SW17.S: now also D39.2 (A)
- net COL9: now reaches SW17.S2
- net COL9: now also SW18.S2, U3.28 (GPA7)
- net COL1: now reaches SW1.1
- net COL1: now also SW9.1, U3.1 (GPB0)
- net at SW1.2: now also D30.2 (A)
- net at D20.2 (A): now also R4.1
- net at D18.2 (A): now also R2.1
- net at D8.1 (DOUT): now also D9.3 (DIN)
- net COL6: now reaches SW14.1
- net COL6: now also SW6.1, U3.6 (GPB5)
- net at SW14.2: now also D27.2 (A)
- net at D4.1 (DOUT): now also D5.3 (DIN)
- net at D4.3 (DIN): now also D3.1 (DOUT)
- net COL2: now reaches SW10.1
- net COL2: now also SW2.1, U3.2 (GPB1)
- net at SW10.2: now also D23.2 (A)
- net at SW6.2: now also D35.2 (A)
- net COL3: now reaches SW11.1
- net COL3: now also SW3.1, U3.3 (GPB2)
- net at SW11.2: now also D24.2 (A)
- net at D14.3 (DIN): now also D13.1 (DOUT)
- net at U1.1 (GPIO26/ADC0/A0): now also D1.3 (DIN)
- net at U1.10 (GPIO4/MISO): now also R2.2
- net at U1.11 (GPIO3/MOSI): now also R1.2
- net +3.3V: now reaches U1.12 (3V3)
- net +3.3V: now also Brd1.1 (VCC)
- net at U1.2 (GPIO27/ADC1/A1): now also J1.3 (Pin_3)
- net at U1.3 (GPIO28/ADC2/A2): now also J1.2 (Pin_2)
- net at U1.4 (GPIO29/ADC3/A3): now also J1.1 (Pin_1)
- net SDA: now reaches U1.5 (GPIO6/SDA)
- net SDA: now also Brd1.4 (SDA), J2.1 (Pin_1), U3.13 (SDA)
- net SCL: now reaches U1.6 (GPIO7/SCL)
- net SCL: now also Brd1.3 (SCL), J2.2 (Pin_2), U3.12 (SCK)
- net at U1.7 (GPIO0/TX): now also R5.2
- net at U1.8 (GPIO1/RX): now also R4.2
- net at U1.9 (GPIO2/SCK): now also R3.2
- net at D13.3 (DIN): now also D12.1 (DOUT)
- net COL5: now reaches SW13.1
- net COL5: now also SW5.1, U3.5 (GPB4)
- net at SW13.2: now also D26.2 (A)
- net at SW2.2: now also D31.2 (A)
- net at D21.2 (A): now also R5.1
- net at D1.1 (DOUT): now also D2.3 (DIN)
- net COL8: now reaches SW16.1
- net COL8: now also SW8.1, U3.8 (GPB7)
- net at SW16.2: now also D29.2 (A)
- net at D6.3 (DIN): now also D5.1 (DOUT)
- net at SW9.2: now also D22.2 (A)
- net COL4: now reaches SW12.1
- net COL4: now also SW4.1, U3.4 (GPB3)
- net at SW12.2: now also D25.2 (A)
- net at SW3.2: now also D32.2 (A)
- net at D17.2 (A): now also R1.1
- net at D2.1 (DOUT): now also D3.3 (DIN)
- net at SW8.2: now also D37.2 (A)
- net SW18.A: now reaches SW18.A
- net SW18.A: now also U3.26 (GPA5)
- net SW18.B: now reaches SW18.B
- net SW18.B: now also U3.27 (GPA6)
- net SW18.S: now reaches SW18.S1
- net SW18.S: now also D38.2 (A)
- net at D19.2 (A): now also R3.1
- net at SW4.2: now also D33.2 (A)
- net COL7: now reaches SW15.1
- net COL7: now also SW7.1, U3.7 (GPB6)
- net at SW15.2: now also D28.2 (A)
- net at SW7.2: now also D36.2 (A)
- net at D11.1 (DOUT): now also D12.3 (DIN)
- net at SW5.2: now also D34.2 (A)
- new net ROW1: D22.1 (K), D23.1 (K), D24.1 (K), D25.1 (K), D26.1 (K), D27.1 (K), D28.1 (K), D29.1 (K), D39.1 (K), U3.21 (GPA0)
- new net ROW2: D30.1 (K), D31.1 (K), D32.1 (K), D33.1 (K), D34.1 (K), D35.1 (K), D36.1 (K), D37.1 (K), D38.1 (K), U3.22 (GPA1)
Other:
- moved on the sheet: D10, D11, D12, D13, D14, D15, D16, D17, D18, D19, D20, D21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

Commit message: Refactor code structure for improved readability and maintainability
Other:
- company: (none) -> @Apfelholz
- title: (none) -> KiCad-Diynamic-Project-Disply-Modul
Changed lines of the file:
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@@
 	(generator_version "9.0")
 	(paper "A4")
+	(title_block
+		(title "KiCad-Diynamic-Project-Disply-Modul")
+		(date "2025-12-14")
+		(rev "1.0")
+		(company "@Apfelholz")
+		(comment 1 "This project implements a custom RP2040-based macro pad.")
+		(comment 2 "It is designed as a programmable input and status device.")
+	)
 	(junction
 		(at 146.05 193.04)
